Commit message: URDF文件修改提交

File: src/mr1000_dual_fr3_description/urdf/dual_fr3_moveit.urdf.xacro (robot description, xacro)
@@ -1,9 +1,4 @@
 <?xml version='1.0' encoding='utf-8'?>
 <robot xmlns:xacro="http://www.ros.org/wiki/xacro" name="dual_fr3">
-    <xacro:arg name="use_fake_hardware" default="true" />
-    <xacro:arg name="fake_sensor_commands" default="false" />
-    <xacro:arg name="gazebo" default="false" />
-    <xacro:arg name="robot_ip_left" default="172.16.0.2" />
-    <xacro:arg name="robot_ip_right" default="172.16.0.3" />
     <xacro:arg name="hand" default="true" />
     <xacro:include filename="$(find mr1000_dual_fr3_description)/urdf/mr1000_macro.xacro" />
@@ -12,5 +7,4 @@
     <xacro:include filename="$(find franka_description)/end_effectors/common/franka_hand.xacro"/>
     <xacro:include filename="$(find franka_description)/end_effectors/common/utils.xacro" />
-    <xacro:include filename="$(find franka_description)/robots/common/franka_arm.ros2_control.xacro"/>
     <xacro:property name="joint_limits" value="${xacro.load_yaml('$(find franka_description)/robots/fr3/joint_limits.yaml')}" />
     <xacro:property name="inertials" value="${xacro.load_yaml('$(find franka_description)/robots/fr3/inertials.yaml')}" />
@@ -25,4 +19,5 @@
         <origin xyz="0 0 0" rpy="0 0 0" />
     </joint>
+    <!-- LEFT ARM -->
     <xacro:franka_arm
         arm_id="fr3"
@@ -30,5 +25,5 @@
         connected_to=""
         safety_distance="0.03"
-        gazebo="$(arg gazebo)"
+        gazebo="false"
         joint_limits="${joint_limits}"
         kinematics="${kinematics}"
@@ -44,22 +39,14 @@
     <xacro:if value="$(arg hand)">
         <xacro:franka_hand
-        connected_to="left_fr3_link8"
-        arm_id="fr3"
-        arm_prefix="left_"
-        ee_id="franka_hand_white"
-        ee_inertials="${hand_inertials}"
-        safety_distance="0.03"
-        gazebo="$(arg gazebo)"
+            connected_to="left_fr3_link8"
+            arm_id="fr3"
+            arm_prefix="left_"
+            ee_id="franka_hand_white"
+            ee_inertials="${hand_inertials}"
+            safety_distance="0.03"
+            gazebo="false"
         />
     </xacro:if>
-    <xacro:franka_arm_ros2_control
-        arm_id="fr3"
-        arm_prefix="left_"
-        robot_ip="$(arg robot_ip_left)"
-        use_fake_hardware="$(arg use_fake_hardware)"
-        fake_sensor_commands="$(arg fake_sensor_commands)"
-        gazebo="$(arg gazebo)"
-        hand="$(arg hand)"
-    />
+    <!-- RIGHT ARM -->
     <xacro:franka_arm
         arm_id="fr3"
@@ -67,5 +54,5 @@
         connected_to=""
         safety_distance="0.03"
-        gazebo="$(arg gazebo)"
+        gazebo="false"
         joint_limits="${joint_limits}"
         kinematics="${kinematics}"
@@ -81,21 +68,12 @@
     <xacro:if value="$(arg hand)">
         <xacro:franka_hand
-        connected_to="right_fr3_link8"
-        arm_id="fr3"
-        arm_prefix="right_"
-        ee_id="franka_hand_white"
-        ee_inertials="${hand_inertials}"
-        safety_distance="0.03"
-        gazebo="$(arg gazebo)"
+            connected_to="right_fr3_link8"
+            arm_id="fr3"
+            arm_prefix="right_"
+            ee_id="franka_hand_white"
+            ee_inertials="${hand_inertials}"
+            safety_distance="0.03"
+            gazebo="false"
         />
     </xacro:if>
-    <xacro:franka_arm_ros2_control
-        arm_id="fr3"
-        arm_prefix="right_"
-        robot_ip="$(arg robot_ip_right)"
-        use_fake_hardware="$(arg use_fake_hardware)"
-        fake_sensor_commands="$(arg fake_sensor_commands)"
-        gazebo="$(arg gazebo)"
-        hand="$(arg hand)"
-    />
 </robot>

File: src/mr1000_dual_fr3_description/urdf/mr1000_macro.xacro (robot description, xacro)
@@ -3,6 +3,6 @@
      Commit Version: 1.6.0-4-g7f85cfe  Build Version: 1.6.7995.38578
      For more information, please see http://wiki.ros.org/sw_urdf_exporter -->
-<robot  xmlns:xacro="http://ros.org/wiki/xacro" name="mr1000_dual_fr3_descriptionn_macro">
-<xacro:macro name="mr1000_dual_fr3_descriptionn_macro">
+<robot  xmlns:xacro="http://ros.org/wiki/xacro" name="mr1000_dual_fr3_description_macro">
+<xacro:macro name="mr1000_dual_fr3_description_macro">
   <link
     name="base_link">
